File: hardware/devboard/devboard.sch (KiCad schematic (older format))
At the start: 69 parts

Commit message: Work on SRAMBB prototype
Parts:
- removed C? (x9): 68u, symbol Device:CP_Small
- removed J?: Conn_02x18_Odd_Even, Connector_PinHeader_2.54mm:PinHeader_2x18_P2.54mm_Vertical, symbol Connector_Generic:Conn_02x18_Odd_Even
- removed R? (x3): 10k, symbol Device:R_Small_US
- removed R? (x3): 100k, symbol Device:R_Small_US
- removed TP? (x9): TestPoint, TestPoint:TestPoint_Bridge_Pitch2.54mm_Drill1.0mm, symbol Connector:TestPoint
- removed U? (x9): 48LM01-I_SM, SOIJ8_SM_MCH, symbol davinci:48LM01-I_SM
- removed U? (x3): MC74VHCT126ADR2G, SOIC-14_NB_ONS, symbol davinci:MC74VHCT126ADR2G
- added C?: 12, symbol Device:CP_Small
- added D? (x2): D_Small, symbol Device:D_Small
- added R?: R_Small_US, symbol Device:R_Small_US
- added U?: CY62187EV30LL-55BAXI, Package_BGA:BGA-48_8.0x9.0mm_Layout6x8_P0.8mm, symbol davinci:CY62187EV30LL-55BAXI
Connections:
- net PE7 is gone; now on net WDI: U?.9 (PE7)
- net GND: now also C?.2, U?.D1 (VSS), U?.E6 (VSS)
- net PC6: now also TP?.1
- net PC7: now also TP?.1
- net VCC: now also U?.D6 (VCC), U?.E1 (VCC)
- net WDI: no longer U?.35 (PC0)
- net B1_EN renamed MEM1_A0
- net MEM1_A0: now also U?.A3 (A0); no longer TP?.1
- net B2_EN renamed MEM1_A1
- net MEM1_A1: now also U?.A4 (A1); no longer TP?.1
- net B3_EN renamed MEM1_A2
- net MEM1_A2: now also U?.A5 (A2); no longer TP?.1
- net C1_CS renamed MEM1_A3
- net MEM1_A3: now also U?.B3 (A3); no longer TP?.1
- net C2_CS renamed MEM1_A4
- net MEM1_A4: now also U?.B4 (A4); no longer TP?.1
- net C3_CS: no longer names the net of TP?.1
- net C3_CS: no longer U?.46 (PA5)
- net MISO renamed MEM1_A11
- net MEM1_A11: now also U?.H5 (A11); no longer TP?.1
- net MOSI renamed MEM1_A10
- net MEM1_A10: now also U?.H4 (A10); no longer TP?.1
- net PA6 renamed MEM1_A6
- net MEM1_A6: now also U?.C4 (A6)
- net PA7 renamed MEM1_A7
- net MEM1_A7: now also U?.D4 (A7)
- net PB0 renamed MEM1_A8
- net MEM1_A8: now also U?.H2 (A8)
- net PB4 renamed MEM1_A12
- net MEM1_A12: now also U?.G3 (A12)
- net PB5 renamed MEM1_A13
- net MEM1_A13: now also U?.G4 (A13)
- net PB6 renamed MEM1_A14
- net MEM1_A14: now also U?.F3 (A14)
- net PB7 renamed MEM1_A15
- net MEM1_A15: now also U?.F4 (A15)
- net PC1 renamed MEM1_A17
- net MEM1_A17: now also U?.D3 (A17)
- net PC2 renamed MEM1_A18
- net MEM1_A18: now also U?.H1 (A18)
- net PC3 renamed MEM1_A19
- net MEM1_A19: now also U?.G2 (A19)
- net PC4 renamed MEM1_A20
- net MEM1_A20: now also U?.H6 (A20)
- net PC5 renamed MEM1_A21
- net MEM1_A21: now also U?.E3 (A21)
- net PD2 renamed MEM1_~CE1
- net MEM1_~CE1: now also TP?.1, U?.B5 (~CE1)
- net PD3 renamed MEM1_CE2
- net MEM1_CE2: now also TP?.1, U?.A6 (CE2)
- net PD4 renamed MEM1_~OE
- net MEM1_~OE: now also TP?.1, U?.A2 (~OE)
- net PD5 renamed MEM1_~BLE
- net MEM1_~BLE: now also TP?.1, U?.A1 (~BLE)
- net PD6 renamed MEM1_~BHE
- net MEM1_~BHE: now also TP?.1, U?.B2 (~BHE)
- net PD7 renamed MEM1_~WE
- net MEM1_~WE: now also TP?.1, U?.G5 (~WE)
- net PE0 renamed MEM1_IO9
- net MEM1_IO9: now also U?.C1 (IO9)
- net PE1 renamed MEM1_IO10
- net MEM1_IO10: now also U?.C2 (IO10)
- net PE2 renamed MEM1_IO11
- net MEM1_IO11: now also U?.D2 (IO11)
- net PE3 renamed MEM1_IO12
- net MEM1_IO12: now also U?.E2 (IO12)
- net PE4 renamed MEM1_IO13
- net MEM1_IO13: now also U?.F2 (IO13)
- net PE5 renamed MEM1_IO14
- net MEM1_IO14: now also U?.F1 (IO14)
- net PE6 renamed MEM1_IO15
- net MEM1_IO15: now also U?.G1 (IO15)
- net PF0 renamed MEM1_IO5
- net MEM1_IO5: now also U?.F5 (IO5)
- net PF1 renamed MEM1_IO6
- net MEM1_IO6: now also U?.F6 (IO6)
- net PF2 renamed MEM1_IO7
- net MEM1_IO7: now also U?.G6 (IO7)
- net PF3 renamed MEM1_IO8
- net MEM1_IO8: now also U?.B1 (IO8)
- net PG0 renamed MEM1_IO0
- net MEM1_IO0: now also U?.B6 (IO0)
- net PG1 renamed MEM1_IO1
- net MEM1_IO1: now also U?.C5 (IO1)
- net PG2 renamed MEM1_IO2
- net MEM1_IO2: now also U?.C6 (IO2)
- net PG3 renamed MEM1_IO3
- net MEM1_IO3: now also U?.D5 (IO3)
- net PG4 renamed MEM1_IO4
- net MEM1_IO4: now also U?.E5 (IO4)
- net SCK renamed MEM1_A9
- net MEM1_A9: now also U?.H3 (A9); no longer TP?.1
- new net: C?.1, D?.2 (A), R?.2
- new net MEM1_A16: U?.35 (PC0), U?.E4 (A16)
- new net MEM1_A5: U?.46 (PA5), U?.C3 (A5)
- new net VDD: D?.1 (K), D?.1 (K), R?.1
- new net VSUPPLY: D?.2 (A)
Other:
- note added: "The diode drops the 3V3 rail to 3V, and prevents current flowing back into the rail."
- note added: "There are some issues here"
- note removed: "CRITICAL:\nCapacitors must be Tantalum with >40% voltage derate"
- note removed: "Memory Banks"
- moved on the sheet: TP?
