File: hardware/devboard/devboard.sch (KiCad schematic (older format))
At the start: 37 parts

Commit message: Improved supercap circuit
Parts:
- removed TP? (x3): TestPoint, TestPoint:TestPoint_Bridge_Pitch2.54mm_Drill1.0mm, symbol Connector:TestPoint
- added D?: 3, symbol Device:D_Zener
- added J?: Conn_01x04, symbol Connector_Generic:Conn_01x04
- added Q?: Q_NMOS_DGS, symbol Device:Q_NMOS_DGS
- added R?: 40k, symbol Device:R_Small_US
- added R?: R_Small_US, symbol Device:R_Small_US
- C?: value 12 -> 12F, 3V
Connections:
- net PC6 is gone; now on net MEM1_CE2: U?.41 (PC6)
- net PC7 is gone; now on net MEM1_~OE: U?.42 (PC7)
- net GND: now also D?.2 (A), J?.4 (Pin_4), R?.2
- net MEM1_CE2: no longer U?.28 (PD3)
- net MEM1_~OE: no longer U?.29 (PD4)
- net VCC: now also J?.1 (Pin_1)
- net VSUPPLY: now also R?.1, R?.1
- net at C?.1, D?.2 (A): now also D?.1 (K), Q?.1 (D); no longer R?.2
- new net: Q?.3 (S), R?.2
- new net: Q?.2 (G), R?.2
- new net UART_RX: J?.3 (Pin_3), U?.29 (PD4)
- new net UART_TX: J?.2 (Pin_2), U?.28 (PD3)
Other:
- note added: "TODO:\nSerial headers"
- note added: "UART HEADER"
- note removed: "The diode drops the 3V3 rail to 3V, and prevents current flowing back into the rail."
- note removed: "There are some issues here"
- moved on the sheet: C?, TP?

Commit message: Update
Parts:
- removed Q?: Q_NMOS_DGS, symbol Device:Q_NMOS_DGS
- removed R?: 40k, symbol Device:R_Small_US
- removed R?: R_Small_US, symbol Device:R_Small_US
- D2, D4: renamed from D?; value D_Small -> Vf < 0.4 V
- D3: renamed from D?; value 3 -> Vz=3 V
- R5: renamed from R?; value R_Small_US -> 33 R
- gave numbers to parts that had none: 32
Connections:
- net at C8.1, D3.1 (K), D4.2 (A): now also R5.2
Other:
- note added: "3.3-1.6 V tolerant"
- note added: "3.3V"
- moved on the sheet: C8, D3
