File: Payload/_autosave-payload.sch (KiCad schematic (older format))
At the start: 86 parts, among them J1 Conn_ARM_JTAG_SWD_10, J2 Conn_01x02, J3 Conn_01x03, Q1 Q_PMOS_GSD, SW1 SW_SPST, U1 STM32L471RGTx, U2 ISO1541, U3 MAX6371, U4 CY62167EV30LL, U5 CY62167EV30LL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

Commit message: Schematic fixes and routing
Parts:
- removed R13: 100 K, Resistor_SMD:R_0603_1608Metric, symbol Device:R_Small_US
Changed lines of the file:
@@
 Wire Wire Line
 	4800 3550 4800 3650
-Connection ~ 5700 4050
 Wire Wire Line
 	4950 3650 4800 3650
@@
 	8950 13100 9250 13100
 $Comp
-L Device:R_Small_US R13
-U 1 1 6078DA87
-P 5850 3850
-F 0 "R13" H 5750 3800 50  0000 C CNN
-F 1 "100 K" V 5750 3650 50  0000 C CNN
-F 2 "Resistor_SMD:R_0603_1608Metric" H 5850 3850 50  0001 C CNN
-F 3 "~" H 5850 3850 50  0001 C CNN
-	1    5850 3850
-	-1   0    0    -1
-$EndComp
-Wire Wire Line
-	5850 3750 5850 3650
-Wire Wire Line
-	5850 3650 5700 3650
-Connection ~ 5700 3650
-Wire Wire Line
-	5700 4050 5850 4050
-Wire Wire Line
-	5850 4050 5850 3950
-$Comp
 L power:GND #PWR029
