File: Payload/payload.sch (KiCad schematic (older format))
At the start: 85 parts, among them J1 Conn_ARM_JTAG_SWD_10, J2 Conn_01x02, J3 Conn_01x03, Q1 Q_PMOS_GSD, SW1 SW_SPST, U1 STM32L471RGTx, U2 ISO1541, U3 MAX6371, U4 CY62167EV30LL, U5 CY62167EV30LL, U6 CY62167EV30LL, U7 CY62167EV30LL, Y1 8 MHz

Commit message: Reduced BOM to fit, routed
Parts:
- removed C15: 100 nF, Capacitor_SMD:C_0603_1608Metric, symbol Device:C_Small
- removed C2, C3: C_Small, Capacitor_SMD:C_0603_1608Metric, symbol Device:C_Small
- removed J3: Conn_01x03, Connector_Wire:SolderWire-0.75sqmm_1x03_P4.8mm_D1.25mm_OD2.3mm_Relief, symbol Connector_Generic:Conn_01x03
- removed R10: R_Small_US, Resistor_SMD:R_0603_1608Metric, symbol Device:R_Small_US
- removed TP1, TP10, TP11, TP12, TP13, TP14, TP15, TP16, TP17, TP18, TP19, TP2, TP20, TP21, TP22, TP23, TP24, TP25, TP26, TP27, TP28, TP29, TP3, TP30, TP31, TP32, TP33, TP34, TP35, TP36, TP37, TP4, TP5, TP6, TP7, TP8, TP9: TestPoint, TestPoint:TestPoint_Pad_1.0x1.0mm, symbol Connector:TestPoint
- removed U7: CY62167EV30LL, Package_SO:TSOP-I-48_18.4x12mm_P0.5mm, symbol Payload2:CY62167EV30LL
- removed Y1: 8 MHz, Payload2:Crystal_SMD_DiodesIncorporated_FY, symbol Device:Crystal_GND24_Small
- added J3: Conn_01x02, Connector_Wire:SolderWire-0.25sqmm_1x02_P4.5mm_D0.65mm_OD2mm, symbol Connector_Generic:Conn_01x02
- added J4: Conn_01x08, Connector_PinHeader_1.27mm:PinHeader_1x08_P1.27mm_Vertical, symbol Connector_Generic:Conn_01x08
- added J5: Conn_02x13_Counter_Clockwise, Connector_PinHeader_1.27mm:PinHeader_2x13_P1.27mm_Vertical, symbol Connector_Generic:Conn_02x13_Counter_Clockwise
- J2: footprint Connector_Wire:SolderWire-0.75sqmm_1x02_P7mm_D1.25mm_OD3.5mm_Relief -> Connector_Wire:SolderWire-0.25sqmm_1x02_P4.5mm_D0.65mm_OD2mm
Connections:
- net A0: now also J5.1 (Pin_1)
- net A1: now also J5.2 (Pin_2)
- net A10: now also J5.11 (Pin_11)
- net A11: now also J5.12 (Pin_12)
- net A12: now also J5.13 (Pin_13)
- net A13: now also J5.14 (Pin_14)
- net A14: now also J5.15 (Pin_15)
- net A15: now also J5.16 (Pin_16)
- net A16: now also J5.17 (Pin_17)
- net A17: now also J5.18 (Pin_18)
- net A18: now also J5.19 (Pin_19)
- net A19: now also J5.20 (Pin_20)
- net A2: now also J5.3 (Pin_3)
- net A20: now also J5.21 (Pin_21)
- net A3: now also J5.4 (Pin_4)
- net A4: now also J5.5 (Pin_5)
- net A5: now also J5.6 (Pin_6)
- net A6: now also J5.7 (Pin_7)
- net A7: now also J5.8 (Pin_8)
- net A8: now also J5.9 (Pin_9)
- net A9: now also J5.10 (Pin_10)
- net I2C3_SCL: now also J3.1 (Pin_1)
- net I2C3_SDA: now also J3.2 (Pin_2)
- net IO0: now also J4.1 (Pin_1)
- net IO1: now also J4.2 (Pin_2)
- net IO2: now also J4.3 (Pin_3)
- net IO3: now also J4.4 (Pin_4)
- net IO4: now also J4.5 (Pin_5)
- net IO5: now also J4.6 (Pin_6)
- net IO6: now also J4.7 (Pin_7)
- net IO7: now also J4.8 (Pin_8)
- net M1_CE: now also J5.24 (Pin_24)
- net M2_CE: now also J5.23 (Pin_23); no longer U1.53 (PC12)
- net M3_CE: now also U1.53 (PC12), J5.22 (Pin_22); no longer U1.52 (PC11)
- net M4_CE: now also U1.52 (PC11); no longer U1.51 (PC10)
- net ~OE: now also J5.26 (Pin_26)
- net ~WE: now also J5.25 (Pin_25)
- no-connect marks 6 -> 8
Other:
- note removed: "NOTE: Internal RC sufficient for operation,\nthis gains a few percent memory clock."
- moved on the sheet: C1, C10, C11, C12, C13, C14, C4, C5, C6, C7, C8, C9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

Commit message: Update component values and isolator
Parts:
- removed U2: ISO1541, Package_SO:SOIC-8_3.9x4.9mm_P1.27mm, symbol Isolator:ISO1541
- added U2: ISO1540, Package_SO:SOIC-8_3.9x4.9mm_P1.27mm, symbol Isolator:ISO1540
- R1: value R_Small_US -> 200 R
- R23: value R_Small_US -> 100
- R8: value 55 R -> 43 R
Connections:
- net GND: now also U2.4 (GND1), U2.5 (GND2)
- net I2C3_SCL: now also U2.7 (SDA2)
- net I2C3_SDA: now also U2.6 (SCL2)
- net VCC: now also U2.1 (VCC1), U2.8 (VCC2)
- net at R6.2, U1.8 (PC0): now also U2.2 (SDA1)
- net at R5.2, U1.9 (PC1): now also U2.3 (SCL1)
Changed lines of the file:
@@
 P 9000 2500
 F 0 "R23" V 9050 2650 50  0000 C CNN
-F 1 "R_Small_US" V 9050 2200 50  0000 C CNN
+F 1 "100" V 9050 2200 50  0000 C CNN
 F 2 "Resistor_SMD:R_0603_1608Metric" H 9000 2500 50  0001 C CNN
 F 3 "~" H 9000 2500 50  0001 C CNN
@@
 U 1 1 6197148F
 P 9700 2700
-F 0 "R25" V 9800 2750 50  0000 C CNN
+F 0 "R25" V 9900 2550 50  0000 C CNN
 F 1 "100 kR" V 9800 2550 50  0000 C CNN
 F 2 "Resistor_SMD:R_0603_1608Metric" H 9700 2700 50  0001 C CNN
@@
 P 9750 9450
 F 0 "R8" V 9950 9400 50  0000 C CNN
-F 1 "55 R" V 9850 9450 50  0000 C CNN
+F 1 "43 R" V 9850 9450 50  0000 C CNN
 F 2 "Resistor_SMD:R_0603_1608Metric" H 9750 9450 50  0001 C CNN
 F 3 "~" H 9750 9450 50  0001 C CNN
@@
 P 8150 3400
 F 0 "R1" H 8300 3450 50  0000 C CNN
-F 1 "R_Small_US" H 8300 3350 50  0000 C CNN
+F 1 "200 R" H 8300 3350 50  0000 C CNN
 F 2 "Resistor_SMD:R_0603_1608Metric" H 8150 3400 50  0001 C CNN
 F 3 "~" H 8150 3400 50  0001 C CNN
 	1    8150 3400
 	1    0    0    1
-$EndComp
-$Comp
-L Isolator:ISO1541 U2
-U 1 1 60830529
-P 1900 4250
-F 0 "U2" H 1900 4617 50  0000 C CNN
-F 1 "ISO1541" H 1900 4526 50  0000 C CNN
-F 2 "Package_SO:SOIC-8_3.9x4.9mm_P1.27mm" H 1900 3900 50  0001 C CNN
-F 3 "http://www.ti.com/lit/ds/symlink/iso1541.pdf" H 1900 4300 50  0001 C CNN
-	1    1900 4250
-	-1   0    0    -1
 $EndComp
 Wire Wire Line
@@
 Text Label 6750 10000 0    50   ~ 0
 A12
+$Comp
+L Isolator:ISO1540 U2
+U 1 1 609473CC
+P 1900 4250
+F 0 "U2" H 1900 4617 50  0000 C CNN
+F 1 "ISO1540" H 1900 4526 50  0000 C CNN
+F 2 "Package_SO:SOIC-8_3.9x4.9mm_P1.27mm" H 1900 3900 50  0001 C CNN
+F 3 "http://www.ti.com/lit/ds/symlink/iso1541.pdf" H 1900 4300 50  0001 C CNN
+	1    1900 4250
+	-1   0    0    -1
+$EndComp
 Wire Bus Line
 	14100 3600 14100 6350

Commit message: Tweak
Parts:
- R12: value 100 K -> 100 kR
- R23: value 100 -> 100 R
Other:
- note added: "NOTE:\n- Software: STM internal comparator -> sense resistor for quick cutoff if latched\n- Software: Can guaruntee rail -> 0 by sensing comparator low side, or switch GPIO to output and drive low.\n Critical that FET conducting and IO low are exclusive if using that approach."
- note removed: "TODO:\nConsider resistors on testpoints\nGeometrically optimize address and IO pin assignments\nVerify that external supply connects to Vin, not Vcc\nIf space permits double up IO resistors as well\n\nNOTE:\n- Software: STM internal comparator -> sense resistor for quick cutoff if latched\n- Software: Can guaruntee rail -> 0 by sensing comparator low side, or switch GPIO to output and drive low.\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"
- note removed: "Text Template"
- moved on the sheet: C1, C10, C11, C12, C13, C14, C4, C5, C6, C7, C8, C9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
